File: pcb/cheetoPet.kicad_pcb (KiCad board)
At the start: 2 copper layers, 50.2 x 95.2 mm, 104 parts, among them CN2 S2B-ZR-SM2-TF, J1 ER-TFT028A3-4, J2 USB_C_Receptacle_USB2.0_16P, Q1 FS8205A, Q2 BSS138, SW1 BTN, SW2 BTN, SW3 BTN, SW4 BTN, SW5 TS24CA, U1 USBLC6-2SC6, U10 TPS63802DLAR, U11 AT24C32M/TR, U12 LTC2955CDDB-1#TRPBF, U13 AT24C32M/TR, U14 AT24C32M/TR, U2 HX PM2.54-1X5P WT, U3 DW01A, U4 BQ24074RGT, U5 MAX17048G_T10, U6 LSM6DSL, U7 PCF8523T/1,118, U8 ESP32-S3-MINI-1U, U9 WS-003DB, X1 SC-32S32.768kHz20PPM7pF

Commit message: pcb update
Other:
- board text added: "screen goes here!"

Commit message: pcb spreadsheet
Routing:
- net GND: vias 85 -> 84
Other:
- board text added: "404:"
- board text added: "cart not found"
- board text added: "error 404"
- board text added: "no name found"
- board text added: "ok lol"
- board text removed: "pet name here..."
- board text removed: "petCart area"
