File: pcb/cheetoPet.kicad_sch (KiCad schematic)
At the start: 104 parts, among them CN2 S2B-ZR-SM2-TF, J1 ER-TFT028A3-4, J2 USB_C_Receptacle_USB2.0_16P, Q1 FS8205A, Q2 BSS138, SW1 BTN, SW2 BTN, SW3 BTN, SW4 BTN, SW5 TS24CA, U1 USBLC6-2SC6, U10 TPS63802DLAR, U11 AT24C32M/TR, U12 LTC2955CDDB-1#TRPBF, U13 AT24C32M/TR, U14 AT24C32M/TR, U2 HX PM2.54-1X5P WT, U3 DW01A, U4 BQ24074RGT, U5 MAX17048G_T10, U6 LSM6DSL, U7 PCF8523T/1,118, U8 ESP32-S3-MINI-1U, U9 WS-003DB, X1 SC-32S32.768kHz20PPM7pF

Commit message: recon mpu
Connections:
- net +3V3: no longer C16.2, U6.5 (VDDIO), U6.8 (VDD)
- net BAT+: now also C16.2, U6.5 (VDDIO), U6.8 (VDD)
Changed lines of the file:
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@@
 		)
 	)
+	(global_label "BAT+"
+		(shape input)
+		(at 213.36 255.27 0)
+		(fields_autoplaced yes)
+		(effects
+			(font
+				(size 1.27 1.27)
+			)
+			(justify left)
+		)
+		(property "Intersheetrefs" "${INTERSHEET_REFS}"
+			(at 221.2438 255.27 0)
+			(hide yes)
+			(show_name no)
+			(do_not_autoplace no)
+			(effects
+				(font
+					(size 1.27 1.27)
+				)
+				(justify left)
+			)
+		)
+	)
 	(global_label "A"
 		(shape input)
@@
 					(unit 1)
 				)
-			)
-		)
-	)
-	(symbol
-		(lib_id "power:+3V3")
-		(at 213.36 255.27 0)
-		(unit 1)
-		(body_style 1)
-		(exclude_from_sim no)
-		(in_bom yes)
-		(on_board yes)
-		(in_pos_files yes)
-		(dnp no)
-		(property "Reference" "#PWR040"
-			(at 213.36 259.08 0)
-			(hide yes)
-			(show_name no)
-			(do_not_autoplace no)
-			(effects
-				(font
-					(size 1.27 1.27)
-				)
-			)
-		)
-		(property "Value" "+3V3"
-			(at 213.36 251.714 0)
-			(show_name no)
-			(do_not_autoplace no)
-			(effects
-				(font
-					(size 1.27 1.27)
-				)
-			)
-		)
-		(property "Footprint" ""
-			(at 213.36 255.27 0)
-			(hide yes)
-			(show_name no)
-			(do_not_autoplace no)
-			(effects
-				(font
-					(size 1.27 1.27)
-				)
-			)
-		)
-		(property "Datasheet" ""
-			(at 213.36 255.27 0)
-			(hide yes)
-			(show_name no)
-			(do_not_autoplace no)
-			(effects
-				(font
-					(size 1.27 1.27)
-				)
-			)
-		)
-		(property "Description" "Power symbol creates a global label with name \"+3V3\""
-			(at 213.36 255.27 0)
-			(hide yes)
-			(show_name no)
-			(do_not_autoplace no)
-			(effects
-				(font
-					(size 1.27 1.27)
-				)
-			)
-		)
-		(pin "1"
-		)
-		(instances
-			(project "cheetoPet"
-				(path "/2746c69b-027c-4aec-b1d7-a024d4e17723"
-					(reference "#PWR040")
-					(unit 1)
-				)
